File: iris-128b/pcb/iris-128b/iris-128b.kicad_pcb (KiCad board)
At the start: 8 copper layers, 45 x 44.5 mm, 77 parts, among them J1 SEAM8-20-S02.0-X-08-3, J2 Conn_02x40_Row_Letter_First

Commit message: adapter board files
Other:
- board text added: "June 2024 CERN-OHL-P v2"
- board text removed: "Designed by Emma Jacobs June 2024"
Changed lines of the file:
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@@
 		(legacy_teardrops no)
 	)
-	(paper "A4")
+	(paper "USLetter")
+	(title_block
+		(title "Iris-128B")
+		(rev "1.0.0")
+		(company "Deku Lab")
+	)
 	(layers
 		(0 "F.Cu" signal "F.Cu (Minimal routing and GND)")
@@
 		(layer "Edge.Cuts")
 	)
-	(gr_text "Designed by \nEmma Jacobs\nJune 2024"
+	(gr_text "June 2024\nCERN-OHL-P v2"
 		(at 123.25 118.625 0)
 		(layer "B.SilkS")
