File: iris-128b/pcb/iris-128b/iris-128b.kicad_sch (KiCad schematic)
At the start: 39 parts, among them J2 Conn_02x40_Row_Letter_First

Commit message: adapter board files
Other:
- note added: "160 pin connector to thin-film"
- note added: "80 pin molex connector to adapter board"
- note added: "Bypass Capacitors"
- note added: "RHS Intan ICs"
- note removed: "${CURRENT_DATE}"
- note removed: "Add a comment here"
- note removed: "DRAFT - Very early stage of schematic, ignore details."
- note removed: "IRIS 128S"
- note removed: "NOTES"
- note removed: "Not fitted components are marked as"
- note removed: "PRELIMINARY - Close to final schematic."
- company: (none) -> Deku Lab
- title: (none) -> Iris-128B
- moved on the sheet: C1, C10, C11, C12, C13, C14, C15, C16, C17, C18, C19, C2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
